File: Circuits/Narcisa.kicad_sch (KiCad schematic)
At the start: 4 parts, among them U1 RC1602A

Commit message: LCD code
Parts:
- added U2: BT04-E, symbol bluetooth:BT04-E
- gave numbers to parts that had none: 1
Connections:
- net +5V: now also U2.1 (5V)
- net GND: now also U2.3 (GND)
- net at A1.17 (D2): no longer U1.4 (RS)
- net at A1.18 (D3): no longer U1.6 (E)
- net at A1.19 (D4): now also U2.4 (KEY); no longer U1.11 (DB4)
- net at A1.20 (D5): now also U2.5 (RXD); no longer U1.12 (DB5)
- net at A1.21 (D6): now also U2.6 (TXD); no longer U1.13 (DB6)
- net at A1.22 (D7): now also U1.4 (RS); no longer U1.14 (DB7)
- net at A1.23 (D8): now also U1.6 (E)
- net at A1.24 (D9): now also U1.11 (DB4)
- net at A1.25 (D10): now also U1.12 (DB5)
- net at A1.26 (D11): now also U1.13 (DB6)
- net at A1.27 (D12): now also U1.14 (DB7)
Other:
- moved on the sheet: R1, RV1, U1

Commit message: Final Commit
Connections:
- net at U2.4 (KEY): no longer A1.19 (D4)
- net at U2.5 (RXD): now also A1.19 (D4); no longer A1.20 (D5)
- net at U2.6 (TXD): now also A1.20 (D5); no longer A1.21 (D6)
- net at U1.4 (RS): now also A1.21 (D6); no longer A1.22 (D7)
- net at U1.6 (E): now also A1.22 (D7); no longer A1.23 (D8)
- net at U1.11 (DB4): now also A1.23 (D8); no longer A1.24 (D9)
- net at U1.12 (DB5): now also A1.24 (D9); no longer A1.25 (D10)
- net at U1.13 (DB6): now also A1.25 (D10); no longer A1.26 (D11)
- net at U1.14 (DB7): now also A1.26 (D11); no longer A1.27 (D12)
